Commit message: Add joint state publisher to Dockerfile and update launch files
- Added ros-humble-joint-state-publisher to the Dockerfile for enhanced joint state management.
- Created new launch files for tethering and simulation, integrating the joint state publisher into the bringup process.
- Updated existing launch files for improved readability and consistency in package usage.

File: ros2_ws/src/robomaster_description/urdf/gripper.urdf.xacro (robot description, xacro)
@@ -156,8 +156,4 @@
         </geometry>
       </collision>
-    </link>
-    <link name="${tf_prefix}gripper_m_link">
-    </link>
-    <link name="${tf_prefix}gripper_t_link">
     </link>
     <link name="${tf_prefix}gripper_m_link">

File: ros2_ws/src/robomaster_description/urdf/robomaster_ep.urdf.xacro (robot description, xacro)
@@ -21,7 +21,7 @@
   <xacro:intelligent_controller tf_prefix="${tf_prefix}" mount="extension" />
   <!-- arm + gripper + camera disabled for mecanum-base attack config -->
-  <!-- <xacro:arm tf_prefix="${tf_prefix}"/>
+  <xacro:arm tf_prefix="${tf_prefix}"/>
   <xacro:camera tf_prefix="${tf_prefix}" mount="arm" camera_yaw="$(arg camera_yaw)"/>
-  <xacro:gripper tf_prefix="${tf_prefix}"/> -->
+  <xacro:gripper tf_prefix="${tf_prefix}"/>
   <xacro:add_tof index="0" tf_prefix="${tf_prefix}" />
   <xacro:add_tof index="1" tf_prefix="${tf_prefix}" />
