Commit message: Kind of functions, added cameras and detection and drivetrain

File: ros2_ws/src/robomaster_description/urdf/arm.urdf.xacro (robot description, xacro)
@@ -263,6 +263,11 @@
         <origin xyz="0.1417841 0.0321051 -0.1257179" rpy="0 0 0" />
         <mass value="0.009" />
-        <inertia ixx="0.0205056" ixy="0.0021202" ixz="-0.0023248" iyy="0.0097562" iyz="0.0101162"
-          izz="0.0117256" />
+        <!-- Placeholder, not measured. The exported tensor here was physically
+             impossible (principal moments failed the triangle inequality) and
+             ~1000x too large for a 9g part, so Gazebo rejected the whole model.
+             This is a cosmetic linkage that nothing drives; if the arm ever
+             needs real dynamics, re-export this about the link's own centre
+             of mass. -->
+        <inertia ixx="1e-5" ixy="0" ixz="0" iyy="1e-5" iyz="0" izz="1e-5" />
       </inertial>
       <visual name="triangle">

File: ros2_ws/src/robomaster_description/urdf/camera.urdf.xacro (robot description, xacro)
@@ -1,5 +1,5 @@
 <?xml version="1.0"?>
 <robot xmlns:xacro="http://playerstage.sourceforge.net/gazebo/xmlschema/#xacro">
-  <xacro:macro name="camera" params="tf_prefix='' mount='' camera_yaw=0.0">
+  <xacro:macro name="camera" params="tf_prefix='' mount='' camera_yaw=0.0 sim:=false">
     <link name="${tf_prefix}camera_link">
       <inertial>
@@ -50,4 +50,41 @@
       <child link="camera_optical_link"/>
     </joint> -->
+    <!-- Topics match camera_node.py's defaults so apriltag_node can't tell sim
+         from the real stream. On camera_optical_link because Gazebo emits the
+         optical convention (Z forward), which apriltag pose assumes. -->
+    <xacro:if value="${sim}">
+      <!-- sdformat lumps fixed-joint children into their parent, which deletes
+           camera_optical_link. The sensor itself survives that, but its frame
+           doesn't - and apriltag poses are only correct against the optical
+           frame. Verified: without this, `ign sdf -p` emits no
+           <link name='camera_optical_link'>. -->
+      <gazebo reference="${tf_prefix}camera_optical_joint">
+        <preserveFixedJoint>true</preserveFixedJoint>
+        <disableFixedJointLumping>true</disableFixedJointLumping>
+      </gazebo>
+      <gazebo reference="${tf_prefix}camera_optical_link">
+        <sensor name="camera" type="camera">
+          <camera>
+            <!-- ~74 deg, approximating the EP's real stream. Gazebo derives
+                 camera_info from this, so sim needs no calibration. -->
+            <horizontal_fov>1.2915</horizontal_fov>
+            <image>
+              <width>1280</width>
+              <height>720</height>
+              <format>R8G8B8</format>
+            </image>
+            <clip>
+              <near>0.05</near>
+              <far>30.0</far>
+            </clip>
+          </camera>
+          <always_on>1</always_on>
+          <update_rate>30</update_rate>
+          <visualize>false</visualize>
+          <topic>camera/image_raw</topic>
+          <gz_frame_id>${tf_prefix}camera_optical_link</gz_frame_id>
+        </sensor>
+      </gazebo>
+    </xacro:if>
   </xacro:macro>
 </robot>

File: ros2_ws/src/robomaster_description/urdf/gripper.urdf.xacro (robot description, xacro)
@@ -376,5 +376,8 @@
       <limit effort="0" velocity="0" />
     </joint>
-    <joint name="${tf_prefix}gripper_link" type="fixed">
+    <!-- Named _joint, not gripper_link: SDF frame names span links AND joints,
+         so sharing the name with the child link makes Gazebo reject the model
+         ("frame with name[gripper_link] already exists"). URDF alone tolerates it. -->
+    <joint name="${tf_prefix}gripper_joint" type="fixed">
       <origin xyz="0.0002793 -0.027026 0.0001815" rpy="0 0 0" />
       <parent link="${tf_prefix}endpoint_bracket_link" />

File: ros2_ws/src/robomaster_description/urdf/robomaster_ep.urdf.xacro (robot description, xacro)
@@ -10,4 +10,11 @@
   </xacro:if>
   <xacro:arg name="camera_yaw" default="0.0" />
+  <!-- Picks which <ros2_control> block is emitted. See ros2_control.urdf.xacro. -->
+  <xacro:arg name="sim" default="false" />
+  <!-- Empty, never a plausible-looking IP: unset must fail (in bringup.launch.py,
+       or on_init if it gets this far), not silently dial the wrong robot. -->
+  <xacro:arg name="robot_ip" default="" />
+  <xacro:arg name="sim_controllers_file" default="" />
+  <xacro:property name="_sim" value="${'$(arg sim)'.lower() == 'true'}" />
   <xacro:include filename="base.urdf.xacro" />
   <xacro:include filename="arm.urdf.xacro" />
@@ -17,4 +24,5 @@
   <xacro:include filename="extension.urdf.xacro" />
   <xacro:include filename="tof.urdf.xacro" />
+  <xacro:include filename="ros2_control.urdf.xacro" />
   <xacro:base tf_prefix="${tf_prefix}" />
   <xacro:extension tf_prefix="${tf_prefix}" use_rear_extension="true" />
@@ -22,5 +30,5 @@
   <!-- arm + gripper + camera for mecanum-base attack config -->
   <xacro:arm tf_prefix="${tf_prefix}"/>
-  <xacro:camera tf_prefix="${tf_prefix}" mount="arm" camera_yaw="$(arg camera_yaw)"/>
+  <xacro:camera tf_prefix="${tf_prefix}" mount="arm" camera_yaw="$(arg camera_yaw)" sim="${_sim}"/>
   <xacro:gripper tf_prefix="${tf_prefix}"/>
   <xacro:add_tof index="0" tf_prefix="${tf_prefix}" />
@@ -28,3 +36,6 @@
   <xacro:add_tof index="2" tf_prefix="${tf_prefix}" />
   <xacro:add_tof index="3" tf_prefix="${tf_prefix}" />
+  <xacro:ros2_control sim="${_sim}" tf_prefix="${tf_prefix}"
+    robot_ip="$(arg robot_ip)"
+    sim_controllers_file="$(arg sim_controllers_file)" />
 </robot>

File: ros2_ws/src/robomaster_description/urdf/wheel.urdf.xacro (robot description, xacro)
@@ -40,5 +40,7 @@
       <child link="${tf_prefix}${name}_wheel_link" />
       <axis xyz="0 1.0 0" />
-      <limit effort="0" velocity="0" />
+      <!-- Must be non-zero or gz_ros2_control clamps wheel commands to 0.
+           velocity is the SDK's 1000 rpm cap in rad/s; effort is a guess. -->
+      <limit effort="5.0" velocity="104.7" />
     </joint>
   </xacro:macro>
